File: Hardware/Solar Panel Electronics/storage_sch.kicad_sch (KiCad schematic)
At the start: 3 parts

Commit message: Edited the charging circuit, need to resize components
Parts:
- C?: value (none) -> 0.1uF
- C?: value (none) -> 10uF
Changed lines of the file:
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@@
       (effects (font (size 1.27 1.27)) (justify left))
     )
-    (property "Value" "" (id 1) (at 116.6368 98.933 0)
+    (property "Value" "0.1uF" (id 1) (at 116.6368 98.933 0)
       (effects (font (size 1.27 1.27)) (justify left))
     )
@@
       (effects (font (size 1.27 1.27)) hide)
     )
-    (property "Value" "" (id 1) (at 132.08 87.63 0))
+    (property "Value" "+3.3V" (id 1) (at 132.08 87.63 0))
     (property "Footprint" "" (id 2) (at 132.08 92.71 0)
       (effects (font (size 1.27 1.27)) hide)
@@
       (effects (font (size 1.27 1.27)) (justify left))
     )
-    (property "Value" "" (id 1) (at 125.5268 98.933 0)
+    (property "Value" "10uF" (id 1) (at 125.5268 98.933 0)
       (effects (font (size 1.27 1.27)) (justify left))
     )

Commit message: Components sized for our requirements. Added ideal diode IC LTC4411 which is more efficient than a normal diode.
Parts:
- gave numbers to parts that had none: 3
Changed lines of the file:
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@@
   (symbol (lib_id "Device:C_Small") (at 114.3 97.79 0) (unit 1)
     (in_bom yes) (on_board yes)
-    (property "Reference" "C?" (id 0) (at 116.6368 96.6216 0)
+    (property "Reference" "C19" (id 0) (at 116.6368 96.6216 0)
       (effects (font (size 1.27 1.27)) (justify left))
     )
@@
   (symbol (lib_id "power:GND") (at 132.08 104.14 0) (unit 1)
     (in_bom yes) (on_board yes)
-    (property "Reference" "#PWR?" (id 0) (at 132.08 110.49 0)
+    (property "Reference" "#PWR0132" (id 0) (at 132.08 110.49 0)
       (effects (font (size 1.27 1.27)) hide)
     )
@@
   (symbol (lib_id "power:GND") (at 187.96 110.49 0) (unit 1)
     (in_bom yes) (on_board yes)
-    (property "Reference" "#PWR?" (id 0) (at 187.96 116.84 0)
+    (property "Reference" "#PWR0133" (id 0) (at 187.96 116.84 0)
       (effects (font (size 1.27 1.27)) hide)
     )
@@
   (symbol (lib_id "power:GND") (at 114.3 102.87 0) (unit 1)
     (in_bom yes) (on_board yes)
-    (property "Reference" "#PWR?" (id 0) (at 114.3 109.22 0)
+    (property "Reference" "#PWR0134" (id 0) (at 114.3 109.22 0)
       (effects (font (size 1.27 1.27)) hide)
     )
@@
   (symbol (lib_id "power:+3.3V") (at 132.08 92.71 0) (unit 1)
     (in_bom yes) (on_board yes) (fields_autoplaced)
-    (property "Reference" "#PWR?" (id 0) (at 132.08 96.52 0)
+    (property "Reference" "#PWR0135" (id 0) (at 132.08 96.52 0)
       (effects (font (size 1.27 1.27)) hide)
     )
@@
   (symbol (lib_id "Device:C_Small") (at 123.19 97.79 0) (unit 1)
     (in_bom yes) (on_board yes)
-    (property "Reference" "C?" (id 0) (at 125.5268 96.6216 0)
+    (property "Reference" "C20" (id 0) (at 125.5268 96.6216 0)
       (effects (font (size 1.27 1.27)) (justify left))
     )
@@
   (symbol (lib_id "Connector:Micro_SD_Card") (at 166.37 93.98 0) (unit 1)
     (in_bom yes) (on_board yes)
-    (property "Reference" "J?" (id 0) (at 165.1 75.7682 0))
+    (property "Reference" "J7" (id 0) (at 165.1 75.7682 0))
     (property "Value" "~" (id 1) (at 165.1 78.0796 0))
     (property "Footprint" "" (id 2) (at 195.58 86.36 0)

Commit message: Assigned Footprints (preliminary - just to do a quick layout)
Parts:
- J7: value ~ -> (none)
Changed lines of the file:
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@@
     (in_bom yes) (on_board yes)
     (property "Reference" "J7" (id 0) (at 165.1 75.7682 0))
-    (property "Value" "~" (id 1) (at 165.1 78.0796 0))
+    (property "Value" "" (id 1) (at 165.1 78.0796 0))
     (property "Footprint" "" (id 2) (at 195.58 86.36 0)
       (effects (font (size 1.27 1.27)) hide)

Commit message: Add Antenna
Parts:
- C19, C20: footprint (none) -> Capacitor_SMD:C_0603_1608Metric
- J7: value (none) -> ~; footprint (none) -> Connector_Card:microSD_HC_Hirose_DM3AT-SF-PEJM5
Changed lines of the file:
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@@
       (effects (font (size 1.27 1.27)) (justify left))
     )
-    (property "Footprint" "" (id 2) (at 114.3 97.79 0)
+    (property "Footprint" "Capacitor_SMD:C_0603_1608Metric" (id 2) (at 114.3 97.79 0)
       (effects (font (size 1.27 1.27)) hide)
     )
@@
       (effects (font (size 1.27 1.27)) (justify left))
     )
-    (property "Footprint" "" (id 2) (at 123.19 97.79 0)
+    (property "Footprint" "Capacitor_SMD:C_0603_1608Metric" (id 2) (at 123.19 97.79 0)
       (effects (font (size 1.27 1.27)) hide)
     )
@@
     (in_bom yes) (on_board yes)
     (property "Reference" "J7" (id 0) (at 165.1 75.7682 0))
-    (property "Value" "" (id 1) (at 165.1 78.0796 0))
-    (property "Footprint" "" (id 2) (at 195.58 86.36 0)
+    (property "Value" "~" (id 1) (at 165.1 78.0796 0))
+    (property "Footprint" "Connector_Card:microSD_HC_Hirose_DM3AT-SF-PEJM5" (id 2) (at 195.58 86.36 0)
       (effects (font (size 1.27 1.27)) hide)
     )

Commit message: Started pcb layout
Parts:
- J7: footprint Connector_Card:microSD_HC_Hirose_DM3AT-SF-PEJM5 -> Connector_Card:microSD_HC_Wuerth_693072010801
Changed lines of the file:
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@@
     (property "Reference" "J7" (id 0) (at 165.1 75.7682 0))
     (property "Value" "~" (id 1) (at 165.1 78.0796 0))
-    (property "Footprint" "Connector_Card:microSD_HC_Hirose_DM3AT-SF-PEJM5" (id 2) (at 195.58 86.36 0)
+    (property "Footprint" "Connector_Card:microSD_HC_Wuerth_693072010801" (id 2) (at 195.58 86.36 0)
       (effects (font (size 1.27 1.27)) hide)
     )
