File: Hardware/Solar Panel Electronics/VoltageReg.kicad_sch (KiCad schematic)
At the start: 32 parts, among them J14 Screw_Terminal_5VRail, Q2 Q_NMOS_DGS, Q3 Q_NMOS_DGS, U6 LM5118MH, U7 LT1963AxST-3.3

Commit message: Need to do routing.
Parts:
- C26: value (none) -> 55nF
- C27: value (none) -> 0.01nF
- R37: value (none) -> 17k
Changed lines of the file:
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@@
     (in_bom yes) (on_board yes) (fields_autoplaced)
     (property "Reference" "R37" (id 0) (at 100.33 90.17 90))
-    (property "Value" "" (id 1) (at 100.33 92.71 90))
+    (property "Value" "17k" (id 1) (at 100.33 92.71 90))
     (property "Footprint" "Resistor_SMD:R_0603_1608Metric" (id 2) (at 100.33 96.52 0)
       (effects (font (size 1.27 1.27)) hide)
@@
     (in_bom yes) (on_board yes) (fields_autoplaced)
     (property "Reference" "C26" (id 0) (at 93.98 88.9 90))
-    (property "Value" "" (id 1) (at 93.98 91.44 90))
+    (property "Value" "55nF" (id 1) (at 93.98 91.44 90))
     (property "Footprint" "Capacitor_SMD:C_0603_1608Metric" (id 2) (at 90.17 97.4852 0)
       (effects (font (size 1.27 1.27)) hide)
@@
     (in_bom yes) (on_board yes) (fields_autoplaced)
     (property "Reference" "C27" (id 0) (at 96.52 93.98 90))
-    (property "Value" "" (id 1) (at 96.52 96.52 90))
+    (property "Value" "0.01nF" (id 1) (at 96.52 96.52 90))
     (property "Footprint" "Capacitor_SMD:C_0603_1608Metric" (id 2) (at 92.71 102.5652 0)
       (effects (font (size 1.27 1.27)) hide)

Commit message: ICARUS v2
Parts:
- removed J14: Screw_Terminal_5VRail, TerminalBlock_TE-Connectivity:TerminalBlock_TE_282834-2_1x02_P2.54mm_Horizontal, symbol Connector:Screw_Terminal_01x02
Changed lines of the file:
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@@
   (junction (at 209.55 91.44) (diameter 0) (color 0 0 0 0)
   )
-  (junction (at 142.24 76.2) (diameter 0) (color 0 0 0 0)
-  )
   (junction (at 107.95 93.98) (diameter 0) (color 0 0 0 0)
   )
@@
     (stroke (width 0) (type default) (color 0 0 0 0))
   )
-  (wire (pts (xy 142.24 76.2) (xy 148.59 76.2))
+  (wire (pts (xy 135.89 76.2) (xy 148.59 76.2))
     (stroke (width 0) (type default) (color 0 0 0 0))
   )
@@
     (stroke (width 0) (type default) (color 0 0 0 0))
   )
-  (wire (pts (xy 142.24 76.2) (xy 142.24 34.29))
-    (stroke (width 0) (type default) (color 0 0 0 0))
-  )
   (wire (pts (xy 69.85 86.36) (xy 83.82 86.36))
     (stroke (width 0) (type default) (color 0 0 0 0))
   )
-  (wire (pts (xy 175.26 36.83) (xy 175.26 43.18))
-    (stroke (width 0) (type default) (color 0 0 0 0))
-  )
   (wire (pts (xy 123.19 54.61) (xy 123.19 76.2))
     (stroke (width 0) (type default) (color 0 0 0 0))
@@
     (stroke (width 0) (type default) (color 0 0 0 0))
   )
-  (wire (pts (xy 181.61 36.83) (xy 175.26 36.83))
-    (stroke (width 0) (type default) (color 0 0 0 0))
-  )
   (wire (pts (xy 29.21 86.36) (xy 29.21 88.9))
     (stroke (width 0) (type default) (color 0 0 0 0))
@@
     (stroke (width 0) (type default) (color 0 0 0 0))
   )
-  (wire (pts (xy 142.24 34.29) (xy 181.61 34.29))
-    (stroke (width 0) (type default) (color 0 0 0 0))
-  )
   (wire (pts (xy 95.25 76.2) (xy 99.06 76.2))
     (stroke (width 0) (type default) (color 0 0 0 0))
@@
   )
   (wire (pts (xy 38.1 66.04) (xy 95.25 66.04))
-    (stroke (width 0) (type default) (color 0 0 0 0))
-  )
-  (wire (pts (xy 135.89 76.2) (xy 142.24 76.2))
     (stroke (width 0) (type default) (color 0 0 0 0))
   )
@@
     )
     (pin "1")
-  )
-  (symbol (lib_id "Connector:Screw_Terminal_01x02") (at 186.69 34.29 0) (unit 1)
-    (in_bom yes) (on_board yes) (fields_autoplaced)
-    (property "Reference" "J14" (id 0) (at 189.23 34.2899 0)
-      (effects (font (size 1.27 1.27)) (justify left))
-    )
-    (property "Value" "Screw_Terminal_5VRail" (id 1) (at 189.23 36.8299 0)
-      (effects (font (size 1.27 1.27)) (justify left))
-    )
-    (property "Footprint" "TerminalBlock_TE-Connectivity:TerminalBlock_TE_282834-2_1x02_P2.54mm_Horizontal" (id 2) (at 186.69 34.29 0)
-      (effects (font (size 1.27 1.27)) hide)
-    )
-    (property "Datasheet" "~" (id 3) (at 186.69 34.29 0)
-      (effects (font (size 1.27 1.27)) hide)
-    )
-    (pin "1")
-    (pin "2")
   )
   (symbol (lib_id "power:GND") (at 135.89 99.06 0) (unit 1)
@@
       (effects (font (size 1.27 1.27)) hide)
     )
-    (pin "1")
-  )
-  (symbol (lib_id "power:GND") (at 175.26 43.18 0) (unit 1)
-    (in_bom yes) (on_board yes) (fields_autoplaced)
-    (property "Reference" "#PWR0138" (id 0) (at 175.26 49.53 0)
-      (effects (font (size 1.27 1.27)) hide)
-    )
-    (property "Value" "GND" (id 1) (at 175.26 48.26 0))
-    (property "Footprint" "" (id 2) (at 175.26 43.18 0)
-      (effects (font (size 1.27 1.27)) hide)
-    )
-    (property "Datasheet" "" (id 3) (at 175.26 43.18 0)
-      (effects (font (size 1.27 1.27)) hide)
-    )

Commit message: final?
Parts:
- L2: footprint Inductor_SMD:L_0603_1608Metric -> Inductor_SMD:L_0805_2012Metric
- R38: value 900 -> 1000
- R39: value 300 -> 332
Connections:
- net GND: now also U6.21 (EP)
Changed lines of the file:
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@@
+    (stroke (width 0) (type default) (color 0 0 0 0))
+  )
+  (wire (pts (xy 59.69 101.6) (xy 59.69 102.2858))
     (stroke (width 0) (type default) (color 0 0 0 0))
   )
@@
     )
     (property "Datasheet" "" (id 3) (at 128.27 67.31 0)
+      (effects (font (size 1.27 1.27)) hide)
+    )
+    (pin "1")
+  )
+  (symbol (lib_id "power:GND") (at 59.69 102.2858 0) (unit 1)
+    (in_bom yes) (on_board yes) (fields_autoplaced)
+    (property "Reference" "#PWR0157" (id 0) (at 59.69 108.6358 0)
+      (effects (font (size 1.27 1.27)) hide)
+    )
+    (property "Value" "GND" (id 1) (at 59.69 107.3658 0))
+    (property "Footprint" "" (id 2) (at 59.69 102.2858 0)
+      (effects (font (size 1.27 1.27)) hide)
+    )
+    (property "Datasheet" "" (id 3) (at 59.69 102.2858 0)
       (effects (font (size 1.27 1.27)) hide)
     )
@@
   (symbol (lib_id "Device:R_Small") (at 135.89 96.52 0) (unit 1)
     (in_bom yes) (on_board yes) (fields_autoplaced)
-    (property "Reference" "R39" (id 0) (at 138.43 95.2499 0)
-      (effects (font (size 1.27 1.27)) (justify left))
-    )
-    (property "Value" "300" (id 1) (at 138.43 97.7899 0)
+    (property "Reference" "R39" (id 0) (at 137.3886 95.6853 0)
+      (effects (font (size 1.27 1.27)) (justify left))
+    )
+    (property "Value" "332" (id 1) (at 137.3886 98.2222 0)
       (effects (font (size 1.27 1.27)) (justify left))
     )
@@
   (symbol (lib_id "Device:R_Small") (at 135.89 91.44 0) (unit 1)
     (in_bom yes) (on_board yes) (fields_autoplaced)
-    (property "Reference" "R38" (id 0) (at 138.43 90.1699 0)
-      (effects (font (size 1.27 1.27)) (justify left))
-    )
-    (property "Value" "900" (id 1) (at 138.43 92.7099 0)
+    (property "Reference" "R38" (id 0) (at 137.3886 90.6053 0)
+      (effects (font (size 1.27 1.27)) (justify left))
+    )
+    (property "Value" "1000" (id 1) (at 137.3886 93.1422 0)
       (effects (font (size 1.27 1.27)) (justify left))
     )
@@
     (property "Reference" "L2" (id 0) (at 102.87 69.85 90))
     (property "Value" "17uH" (id 1) (at 102.87 72.39 90))
-    (property "Footprint" "Inductor_SMD:L_0603_1608Metric" (id 2) (at 102.87 76.2 0)
-      (effects (font (size 1.27 1.27)) hide)
-    )
+    (property "Footprint" "Inductor_SMD:L_0805_2012Metric" (id 2) (at 102.87 76.2 0)
+      (effects (font (size 1.27 1.27)) hide)
+    )
