File: Hardware/Solar Panel Electronics/usbToUart.kicad_sch (KiCad schematic)
At the start: 17 parts, among them J6 USB_C_Receptacle_USB2.0, U5 INTERFACE-CP2102-GMR(QFN28)

Commit message: final?
Parts:
- removed C15: 4.7uF, Capacitor_SMD:CP_Elec_3x5.3, symbol Device:CP1_Small
- added C15: 47uF, Capacitor_SMD:C_0603_1608Metric, symbol Device:C_Small
Connections:
- net +3V3: now also C15.2
- net GND: now also U5.29 (GND@1), C15.1
- no-connect marks 20 -> 19
Changed lines of the file:
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@@
   (junction (at 160.02 80.01) (diameter 0) (color 0 0 0 0)
   )
+  (junction (at 144.7292 77.47) (diameter 0) (color 0 0 0 0)
+  )
   (junction (at 158.75 77.47) (diameter 0) (color 0 0 0 0)
   )
@@
   )
   (junction (at 124.46 67.31) (diameter 0) (color 0 0 0 0)
-  )
-  (junction (at 144.78 77.47) (diameter 0) (color 0 0 0 0)
   )
   (junction (at 154.94 88.9) (diameter 0) (color 0 0 0 0)
@@
   (no_connect (at 208.28 64.77))
   (no_connect (at 167.64 64.77))
-  (no_connect (at 177.8 52.07))
   (no_connect (at 182.88 52.07))
   (no_connect (at 114.3 87.63))
@@
     (stroke (width 0) (type default) (color 0 0 0 0))
   )
+  (wire (pts (xy 173.736 50.4952) (xy 173.736 49.784))
+    (stroke (width 0) (type default) (color 0 0 0 0))
+  )
   (wire (pts (xy 116.84 69.85) (xy 119.38 69.85))
     (stroke (width 0) (type default) (color 0 0 0 0))
@@
     (stroke (width 0) (type default) (color 0 0 0 0))
   )
+  (wire (pts (xy 144.7292 71.0946) (xy 144.7292 69.85))
+    (stroke (width 0) (type default) (color 0 0 0 0))
+  )
   (wire (pts (xy 124.46 69.85) (xy 124.46 67.31))
     (stroke (width 0) (type default) (color 0 0 0 0))
@@
     (stroke (width 0) (type default) (color 0 0 0 0))
   )
-  (wire (pts (xy 144.78 76.2) (xy 144.78 77.47))
+  (wire (pts (xy 173.736 49.784) (xy 177.8 49.784))
     (stroke (width 0) (type default) (color 0 0 0 0))
   )
@@
     (stroke (width 0) (type default) (color 0 0 0 0))
   )
-  (wire (pts (xy 158.75 77.47) (xy 144.78 77.47))
+  (wire (pts (xy 137.16 77.47) (xy 144.7292 77.47))
     (stroke (width 0) (type default) (color 0 0 0 0))
   )
@@
     (stroke (width 0) (type default) (color 0 0 0 0))
   )
-  (wire (pts (xy 144.78 71.12) (xy 144.78 69.85))
-    (stroke (width 0) (type default) (color 0 0 0 0))
-  )
   (wire (pts (xy 207.01 118.11) (xy 204.47 118.11))
     (stroke (width 0) (type default) (color 0 0 0 0))
@@
     (stroke (width 0) (type default) (color 0 0 0 0))
   )
-  (wire (pts (xy 144.78 69.85) (xy 158.75 69.85))
+  (wire (pts (xy 177.8 49.784) (xy 177.8 52.07))
+    (stroke (width 0) (type default) (color 0 0 0 0))
+  )
+  (wire (pts (xy 144.7292 69.85) (xy 158.75 69.85))
     (stroke (width 0) (type default) (color 0 0 0 0))
   )
@@
     (stroke (width 0) (type default) (color 0 0 0 0))
   )
-  (wire (pts (xy 137.16 77.47) (xy 144.78 77.47))
-    (stroke (width 0) (type default) (color 0 0 0 0))
-  )
   (wire (pts (xy 124.46 67.31) (xy 125.73 67.31))
     (stroke (width 0) (type default) (color 0 0 0 0))
@@
   )
   (wire (pts (xy 170.18 102.87) (xy 180.34 102.87))
+    (stroke (width 0) (type default) (color 0 0 0 0))
+  )
+  (wire (pts (xy 144.7292 76.1746) (xy 144.7292 77.47))
+    (stroke (width 0) (type default) (color 0 0 0 0))
+  )
+  (wire (pts (xy 144.7292 77.47) (xy 158.75 77.47))
     (stroke (width 0) (type default) (color 0 0 0 0))
   )
@@
   (hierarchical_label "RXD" (shape output) (at 187.96 44.45 90)
     (effects (font (size 1.27 1.27)) (justify left))
-  )
-  (symbol (lib_id "Device:CP1_Small") (at 144.78 73.66 180) (unit 1)
-    (in_bom yes) (on_board yes)
-    (property "Reference" "C15" (id 0) (at 142.4686 74.8284 0)
-      (effects (font (size 1.27 1.27)) (justify left))
-    )
-    (property "Value" "4.7uF" (id 1) (at 142.4686 72.517 0)
-      (effects (font (size 1.27 1.27)) (justify left))
-    )
-    (property "Footprint" "Capacitor_SMD:CP_Elec_3x5.3" (id 2) (at 144.78 73.66 0)
-      (effects (font (size 1.27 1.27)) hide)
-    )
-    (property "Datasheet" "~" (id 3) (at 144.78 73.66 0)
-      (effects (font (size 1.27 1.27)) hide)
-    )
-    (pin "1")
-    (pin "2")
   )
   (symbol (lib_id "power:VBUS") (at 170.18 97.79 0) (unit 1)
@@
     (pin "2")
   )
+  (symbol (lib_id "Device:C_Small") (at 144.7292 73.6346 0) (unit 1)
+    (in_bom yes) (on_board yes) (fields_autoplaced)
+    (property "Reference" "C15" (id 0) (at 147.0533 72.8062 0)
+      (effects (font (size 1.27 1.27)) (justify left))
+    )
+    (property "Value" "47uF" (id 1) (at 147.0533 75.3431 0)
+      (effects (font (size 1.27 1.27)) (justify left))
+    )
+    (property "Footprint" "Capacitor_SMD:C_0603_1608Metric" (id 2) (at 144.7292 73.6346 0)
+      (effects (font (size 1.27 1.27)) hide)
+    )
+    (property "Datasheet" "~" (id 3) (at 144.7292 73.6346 0)
+      (effects (font (size 1.27 1.27)) hide)
+    )
+    (pin "1")
+    (pin "2")
+  )
   (symbol (lib_id "power:GND") (at 212.09 118.11 90) (unit 1)
     (in_bom yes) (on_board yes)
@@
       (effects (font (size 1.27 1.27)) hide)
     )
+    (pin "1")
+  )
+  (symbol (lib_id "power:GND") (at 173.736 50.4952 0) (unit 1)
+    (in_bom yes) (on_board yes)
+    (property "Reference" "#PWR0156" (id 0) (at 173.736 56.8452 0)
+      (effects (font (size 1.27 1.27)) hide)
+    )
+    (property "Value" "GND" (id 1) (at 173.863 53.7464 90)
+      (effects (font (size 1.27 1.27)) (justify right))
+    )
+    (property "Footprint" "" (id 2) (at 173.736 50.4952 0)
+      (effects (font (size 1.27 1.27)) hide)
+    )
+    (property "Datasheet" "" (id 3) (at 173.736 50.4952 0)
+      (effects (font (size 1.27 1.27)) hide)
+    )
