File: Hardware/Solar Panel Electronics/ADC.kicad_sch (KiCad schematic)
At the start: 23 parts

Commit message: Made changes to solar charging circuit
Parts:
- C? (x2): value (none) -> 10uF
- C? (x2): value (none) -> 10nF
- C?: value (none) -> 220nF
- R? (x6), R_Shunt? (x3): value (none) -> 1k
- R?: value (none) -> 10k
- U?: value (none) -> ADS131M04
Changed lines of the file:
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@@
     (in_bom yes) (on_board yes) (fields_autoplaced)
     (property "Reference" "R?" (id 0) (at 106.68 88.9 90))
-    (property "Value" "" (id 1) (at 106.68 91.44 90))
+    (property "Value" "1k" (id 1) (at 106.68 91.44 90))
     (property "Footprint" "" (id 2) (at 106.68 95.25 0)
       (effects (font (size 1.27 1.27)) hide)
@@
     (in_bom yes) (on_board yes) (fields_autoplaced)
     (property "Reference" "R?" (id 0) (at 106.68 109.22 90))
-    (property "Value" "" (id 1) (at 106.68 111.76 90))
+    (property "Value" "1k" (id 1) (at 106.68 111.76 90))
     (property "Footprint" "" (id 2) (at 106.68 115.57 0)
       (effects (font (size 1.27 1.27)) hide)
@@
     (in_bom yes) (on_board yes) (fields_autoplaced)
     (property "Reference" "R?" (id 0) (at 106.68 101.6 90))
-    (property "Value" "" (id 1) (at 106.68 104.14 90))
+    (property "Value" "1k" (id 1) (at 106.68 104.14 90))
     (property "Footprint" "" (id 2) (at 106.68 107.95 0)
       (effects (font (size 1.27 1.27)) hide)
@@
       (effects (font (size 1.27 1.27)) (justify left))
     )
-    (property "Value" "" (id 1) (at 93.98 68.5799 0)
+    (property "Value" "1k" (id 1) (at 93.98 68.5799 0)
       (effects (font (size 1.27 1.27)) (justify left))
     )
@@
       (effects (font (size 1.27 1.27)) (justify left))
     )
-    (property "Value" "" (id 1) (at 93.98 113.0299 0)
+    (property "Value" "1k" (id 1) (at 93.98 113.0299 0)
       (effects (font (size 1.27 1.27)) (justify left))
     )
@@
       (effects (font (size 1.27 1.27)) hide)
     )
-    (property "Value" "" (id 1) (at 198.12 73.66 0))
+    (property "Value" "+3.3V" (id 1) (at 198.12 73.66 0))
     (property "Footprint" "" (id 2) (at 198.12 78.74 0)
       (effects (font (size 1.27 1.27)) hide)
@@
       (effects (font (size 1.27 1.27)) hide)
     )
-    (property "Value" "" (id 1) (at 143.51 78.74 0))
+    (property "Value" "+3.3V" (id 1) (at 143.51 78.74 0))
     (property "Footprint" "" (id 2) (at 143.51 83.82 0)
       (effects (font (size 1.27 1.27)) hide)
@@
       (effects (font (size 1.27 1.27)) (justify right))
     )
-    (property "Value" "" (id 1) (at 146.05 90.1635 0)
+    (property "Value" "10uF" (id 1) (at 146.05 90.1635 0)
       (effects (font (size 1.27 1.27)) (justify right))
     )
@@
       (effects (font (size 1.27 1.27)) (justify right))
     )
-    (property "Value" "" (id 1) (at 210.82 104.14 0)
+    (property "Value" "10k" (id 1) (at 210.82 104.14 0)
       (effects (font (size 1.27 1.27)) (justify right))
     )
@@
       (effects (font (size 1.27 1.27)) (justify left))
     )
-    (property "Value" "" (id 1) (at 114.3 92.7162 0)
+    (property "Value" "10nF" (id 1) (at 114.3 92.7162 0)
       (effects (font (size 1.27 1.27)) (justify left))
     )
@@
     (in_bom yes) (on_board yes) (fields_autoplaced)
     (property "Reference" "R?" (id 0) (at 106.68 57.15 90))
-    (property "Value" "" (id 1) (at 106.68 59.69 90))
+    (property "Value" "1k" (id 1) (at 106.68 59.69 90))
     (property "Footprint" "" (id 2) (at 106.68 63.5 0)
       (effects (font (size 1.27 1.27)) hide)
@@
       (effects (font (size 1.27 1.27)) hide)
     )
-    (property "Value" "" (id 1) (at 91.44 78.74 0))
+    (property "Value" "GND" (id 1) (at 91.44 78.74 0))
     (property "Footprint" "" (id 2) (at 91.44 73.66 0)
       (effects (font (size 1.27 1.27)) hide)
@@
       (effects (font (size 1.27 1.27)) (justify left))
     )
-    (property "Value" "" (id 1) (at 114.3 68.5862 0)
+    (property "Value" "10nF" (id 1) (at 114.3 68.5862 0)
       (effects (font (size 1.27 1.27)) (justify left))
     )
@@
       (effects (font (size 1.27 1.27)) (justify left))
     )
-    (property "Value" "" (id 1) (at 93.98 92.7099 0)
+    (property "Value" "1k" (id 1) (at 93.98 92.7099 0)
       (effects (font (size 1.27 1.27)) (justify left))
     )
@@
     (in_bom yes) (on_board yes) (fields_autoplaced)
     (property "Reference" "R?" (id 0) (at 106.68 64.77 90))
-    (property "Value" "" (id 1) (at 106.68 67.31 90))
+    (property "Value" "1k" (id 1) (at 106.68 67.31 90))
     (property "Footprint" "" (id 2) (at 106.68 71.12 0)
       (effects (font (size 1.27 1.27)) hide)
@@
       (effects (font (size 1.27 1.27)) (justify right))
     )
-    (property "Value" "" (id 1) (at 204.47 85.0835 0)
+    (property "Value" "10uF" (id 1) (at 204.47 85.0835 0)
       (effects (font (size 1.27 1.27)) (justify right))
     )
@@
     (in_bom yes) (on_board yes) (fields_autoplaced)
     (property "Reference" "C?" (id 0) (at 193.0336 83.82 90))
-    (property "Value" "" (id 1) (at 193.0336 86.36 90))
+    (property "Value" "220nF" (id 1) (at 193.0336 86.36 90))
     (property "Footprint" "" (id 2) (at 193.04 90.17 0)
       (effects (font (size 1.27 1.27)) hide)
@@
     (in_bom yes) (on_board yes) (fields_autoplaced)
     (property "Reference" "U?" (id 0) (at 175.26 78.74 0))
-    (property "Value" "" (id 1) (at 175.26 81.28 0))
+    (property "Value" "ADS131M04" (id 1) (at 175.26 81.28 0))
     (property "Footprint" "" (id 2) (at 170.18 95.25 0)
       (effects (font (size 1.27 1.27)) hide)
@@
     (in_bom yes) (on_board yes) (fields_autoplaced)
     (property "Reference" "R?" (id 0) (at 106.68 81.28 90))
-    (property "Value" "" (id 1) (at 106.68 83.82 90))
+    (property "Value" "1k" (id 1) (at 106.68 83.82 90))
     (property "Footprint" "" (id 2) (at 106.68 87.63 0)
       (effects (font (size 1.27 1.27)) hide)

Commit message: Changed to use ADS131M04 adc instead of esp32 adc for power calculation
Parts:
- removed C?: ~, symbol Device:C
- removed J?, Patch?: ~, symbol Connector:Screw_Terminal_01x02
- removed JP?: ~, symbol daq-hardware-rescue:Jumper_NO_Small-Device
- removed R?, R_Shunt?: 1k, symbol Device:R_Small
- added C?: ~, symbol Device:C_Small
- added R?: 1k, symbol Device:R_Small
Connections:
- net AIN2N is gone; now on net GND: C?.2, U?.8 (AIN2N)
- net AIN3N is gone; now on net GND: U?.9 (AIN3N)
- net AIN3P: now also C?.1, R?.1
- net GND: now also C?.2
- net MappedVoltage1: now reaches R?.2
- new net MappedVoltage2: R?.2

Commit message: Assigned Footprints (preliminary - just to do a quick layout)
Parts:
- U8: renamed from U?; value ADS131M04 -> (none)
- gave numbers to parts that had none: 18
Changed lines of the file:
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@@
   (symbol (lib_id "Device:R_Small") (at 106.68 95.25 90) (unit 1)
     (in_bom yes) (on_board yes) (fields_autoplaced)
-    (property "Reference" "R?" (id 0) (at 106.68 88.9 90))
+    (property "Reference" "R43" (id 0) (at 106.68 88.9 90))
     (property "Value" "1k" (id 1) (at 106.68 91.44 90))
     (property "Footprint" "" (id 2) (at 106.68 95.25 0)
@@
   (symbol (lib_id "Device:C_Small") (at 111.76 111.76 0) (unit 1)
     (in_bom yes) (on_board yes) (fields_autoplaced)
-    (property "Reference" "C?" (id 0) (at 114.3 110.4962 0)
+    (property "Reference" "C33" (id 0) (at 114.3 110.4962 0)
       (effects (font (size 1.27 1.27)) (justify left))
     )
@@
   (symbol (lib_id "Device:R_Small") (at 106.68 107.95 270) (unit 1)
     (in_bom yes) (on_board yes) (fields_autoplaced)
-    (property "Reference" "R?" (id 0) (at 106.68 101.6 90))
+    (property "Reference" "R44" (id 0) (at 106.68 101.6 90))
     (property "Value" "1k" (id 1) (at 106.68 104.14 90))
     (property "Footprint" "" (id 2) (at 106.68 107.95 0)
@@
   (symbol (lib_id "Device:R_Small") (at 106.68 127 270) (unit 1)
     (in_bom yes) (on_board yes) (fields_autoplaced)
-    (property "Reference" "R?" (id 0) (at 106.68 120.65 90))
+    (property "Reference" "R45" (id 0) (at 106.68 120.65 90))
     (property "Value" "1k" (id 1) (at 106.68 123.19 90))
     (property "Footprint" "" (id 2) (at 106.68 127 0)
@@
   (symbol (lib_id "power:GND") (at 91.44 97.79 0) (unit 1)
     (in_bom yes) (on_board yes) (fields_autoplaced)
-    (property "Reference" "#PWR?" (id 0) (at 91.44 104.14 0)
+    (property "Reference" "#PWR025" (id 0) (at 91.44 104.14 0)
       (effects (font (size 1.27 1.27)) hide)
     )
@@
   (symbol (lib_id "Device:R_Small") (at 91.44 67.31 0) (unit 1)
     (in_bom yes) (on_board yes) (fields_autoplaced)
-    (property "Reference" "R_Shunt?" (id 0) (at 93.98 66.0399 0)
+    (property "Reference" "R_Shunt1" (id 0) (at 93.98 66.0399 0)
       (effects (font (size 1.27 1.27)) (justify left))
     )
@@
   (symbol (lib_id "power:+3.3V") (at 198.12 78.74 0) (unit 1)
     (in_bom yes) (on_board yes) (fields_autoplaced)
-    (property "Reference" "#PWR?" (id 0) (at 198.12 82.55 0)
+    (property "Reference" "#PWR031" (id 0) (at 198.12 82.55 0)
       (effects (font (size 1.27 1.27)) hide)
     )
@@
   (symbol (lib_id "power:+3.3V") (at 143.51 83.82 0) (unit 1)
     (in_bom yes) (on_board yes) (fields_autoplaced)
-    (property "Reference" "#PWR?" (id 0) (at 143.51 87.63 0)
+    (property "Reference" "#PWR028" (id 0) (at 143.51 87.63 0)
       (effects (font (size 1.27 1.27)) hide)
     )
@@
   (symbol (lib_id "power:GND") (at 143.51 92.71 0) (unit 1)
     (in_bom yes) (on_board yes)
-    (property "Reference" "#PWR?" (id 0) (at 143.51 99.06 0)
+    (property "Reference" "#PWR029" (id 0) (at 143.51 99.06 0)
       (effects (font (size 1.27 1.27)) hide)
     )
@@
   (symbol (lib_id "Device:C_Small") (at 143.51 88.9 180) (unit 1)
     (in_bom yes) (on_board yes) (fields_autoplaced)
-    (property "Reference" "C?" (id 0) (at 146.05 87.6235 0)
+    (property "Reference" "C35" (id 0) (at 146.05 87.6235 0)
       (effects (font (size 1.27 1.27)) (justify right))
     )
@@
   (symbol (lib_id "power:GND") (at 121.92 134.62 0) (unit 1)
     (in_bom yes) (on_board yes) (fields_autoplaced)
-    (property "Reference" "#PWR?" (id 0) (at 121.92 140.97 0)
+    (property "Reference" "#PWR027" (id 0) (at 121.92 140.97 0)
       (effects (font (size 1.27 1.27)) hide)
     )
@@
   (symbol (lib_id "Device:R") (at 209.55 102.87 180) (unit 1)
     (in_bom yes) (on_board yes)
-    (property "Reference" "R?" (id 0) (at 211.328 101.7016 0)
+    (property "Reference" "R46" (id 0) (at 211.328 101.7016 0)
       (effects (font (size 1.27 1.27)) (justify right))
     )
@@
   (symbol (lib_id "power:GND") (at 152.4 88.9 0) (unit 1)
     (in_bom yes) (on_board yes)
-    (property "Reference" "#PWR?" (id 0) (at 152.4 95.25 0)
+    (property "Reference" "#PWR030" (id 0) (at 152.4 95.25 0)
       (effects (font (size 1.27 1.27)) hide)
     )
@@
   (symbol (lib_id "Device:C_Small") (at 111.76 91.44 0) (unit 1)
     (in_bom yes) (on_board yes) (fields_autoplaced)
-    (property "Reference" "C?" (id 0) (at 114.3 90.1762 0)
+    (property "Reference" "C32" (id 0) (at 114.3 90.1762 0)
       (effects (font (size 1.27 1.27)) (justify left))
     )
@@
   (symbol (lib_id "power:GND") (at 121.92 115.57 0) (unit 1)
     (in_bom yes) (on_board yes) (fields_autoplaced)
-    (property "Reference" "#PWR?" (id 0) (at 121.92 121.92 0)
+    (property "Reference" "#PWR026" (id 0) (at 121.92 121.92 0)
       (effects (font (size 1.27 1.27)) hide)
     )
@@
   (symbol (lib_id "Device:R_Small") (at 106.68 63.5 270) (unit 1)
     (in_bom yes) (on_board yes) (fields_autoplaced)
-    (property "Reference" "R?" (id 0) (at 106.68 57.15 90))
+    (property "Reference" "R40" (id 0) (at 106.68 57.15 90))
     (property "Value" "1k" (id 1) (at 106.68 59.69 90))
     (property "Footprint" "" (id 2) (at 106.68 63.5 0)
@@
   (symbol (lib_id "power:GND") (at 91.44 73.66 0) (unit 1)
     (in_bom yes) (on_board yes) (fields_autoplaced)
-    (property "Reference" "#PWR?" (id 0) (at 91.44 80.01 0)
+    (property "Reference" "#PWR024" (id 0) (at 91.44 80.01 0)
       (effects (font (size 1.27 1.27)) hide)
     )
@@
   (symbol (lib_id "Device:C_Small") (at 111.76 67.31 0) (unit 1)
     (in_bom yes) (on_board yes) (fields_autoplaced)
-    (property "Reference" "C?" (id 0) (at 114.3 66.0462 0)
+    (property "Reference" "C31" (id 0) (at 114.3 66.0462 0)
       (effects (font (size 1.27 1.27)) (justify left))
     )
@@
   (symbol (lib_id "Device:R_Small") (at 91.44 91.44 0) (unit 1)
     (in_bom yes) (on_board yes) (fields_autoplaced)
-    (property "Reference" "R_Shunt?" (id 0) (at 93.98 90.1699 0)
+    (property "Reference" "R_Shunt2" (id 0) (at 93.98 90.1699 0)
       (effects (font (size 1.27 1.27)) (justify left))
     )
@@
   (symbol (lib_id "Connector:Screw_Terminal_01x02") (at 81.28 90.17 0) (mirror y) (unit 1)
     (in_bom yes) (on_board yes)
-    (property "Reference" "Patch?" (id 0) (at 83.3628 95.885 0))
+    (property "Reference" "Patch2" (id 0) (at 83.3628 95.885 0))
     (property "Value" "~" (id 1) (at 83.3628 93.5736 0))
     (property "Footprint" "" (id 2) (at 81.28 90.17 0)
@@
   (symbol (lib_id "Device:R_Small") (at 106.68 71.12 90) (unit 1)
     (in_bom yes) (on_board yes) (fields_autoplaced)
-    (property "Reference" "R?" (id 0) (at 106.68 64.77 90))
+    (property "Reference" "R41" (id 0) (at 106.68 64.77 90))
     (property "Value" "1k" (id 1) (at 106.68 67.31 90))
     (property "Footprint" "" (id 2) (at 106.68 71.12 0)
@@
   (symbol (lib_id "Connector:Screw_Terminal_01x02") (at 81.28 66.04 0) (mirror y) (unit 1)
     (in_bom yes) (on_board yes)
-    (property "Reference" "Patch?" (id 0) (at 83.3628 71.755 0))
+    (property "Reference" "Patch1" (id 0) (at 83.3628 71.755 0))
     (property "Value" "~" (id 1) (at 83.3628 69.4436 0))
     (property "Footprint" "" (id 2) (at 81.28 66.04 0)
@@
   (symbol (lib_id "Device:C_Small") (at 201.93 83.82 180) (unit 1)
     (in_bom yes) (on_board yes) (fields_autoplaced)
-    (property "Reference" "C?" (id 0) (at 204.47 82.5435 0)
+    (property "Reference" "C37" (id 0) (at 204.47 82.5435 0)
       (effects (font (size 1.27 1.27)) (justify right))
     )
@@
   (symbol (lib_id "power:+3V3") (at 209.55 97.79 0) (unit 1)
     (in_bom yes) (on_board yes)
-    (property "Reference" "#PWR?" (id 0) (at 209.55 101.6 0)
+    (property "Reference" "#PWR033" (id 0) (at 209.55 101.6 0)
       (effects (font (size 1.27 1.27)) hide)
     )
@@
   (symbol (lib_id "Device:C_Small") (at 193.04 90.17 270) (unit 1)
     (in_bom yes) (on_board yes) (fields_autoplaced)
-    (property "Reference" "C?" (id 0) (at 193.0336 83.82 90))
+    (property "Reference" "C36" (id 0) (at 193.0336 83.82 90))
     (property "Value" "220nF" (id 1) (at 193.0336 86.36 90))
     (property "Footprint" "" (id 2) (at 193.04 90.17 0)
@@
   (symbol (lib_id "iclr:ADS131M04") (at 175.26 96.52 0) (unit 1)
     (in_bom yes) (on_board yes) (fields_autoplaced)
-    (property "Reference" "U?" (id 0) (at 175.26 78.74 0))
-    (property "Value" "ADS131M04" (id 1) (at 175.26 81.28 0))
+    (property "Reference" "U8" (id 0) (at 175.26 78.74 0))
+    (property "Value" "" (id 1) (at 175.26 81.28 0))
     (property "Footprint" "" (id 2) (at 170.18 95.25 0)
       (effects (font (size 1.27 1.27)) hide)
@@
   (symbol (lib_id "power:GND") (at 209.55 87.63 0) (unit 1)
     (in_bom yes) (on_board yes)
-    (property "Reference" "#PWR?" (id 0) (at 209.55 93.98 0)
+    (property "Reference" "#PWR032" (id 0) (at 209.55 93.98 0)
       (effects (font (size 1.27 1.27)) hide)
     )
@@
   (symbol (lib_id "Device:C_Small") (at 111.76 130.81 0) (unit 1)
     (in_bom yes) (on_board yes) (fields_autoplaced)
-    (property "Reference" "C?" (id 0) (at 114.3 129.5462 0)
+    (property "Reference" "C34" (id 0) (at 114.3 129.5462 0)
       (effects (font (size 1.27 1.27)) (justify left))
     )
@@
   (symbol (lib_id "Device:R_Small") (at 106.68 87.63 270) (unit 1)
     (in_bom yes) (on_board yes) (fields_autoplaced)
-    (property "Reference" "R?" (id 0) (at 106.68 81.28 90))
+    (property "Reference" "R42" (id 0) (at 106.68 81.28 90))
     (property "Value" "1k" (id 1) (at 106.68 83.82 90))
     (property "Footprint" "" (id 2) (at 106.68 87.63 0)

Commit message: Add Antenna
Parts:
- C31, C32, C33, C34, C35, C36, C37: footprint (none) -> Capacitor_SMD:C_0603_1608Metric
- Patch1, Patch2: footprint (none) -> TerminalBlock_TE-Connectivity:TerminalBlock_TE_282834-2_1x02_P2.54mm_Horizontal
- R40, R41, R42, R43, R44, R45, R46, R_Shunt1, R_Shunt2: footprint (none) -> Resistor_SMD:R_0603_1608Metric
- U8: value (none) -> ADS131M04; footprint (none) -> Package_DFN_QFN:WQFN-20-1EP_3x3mm_P0.4mm_EP1.7x1.7mm_ThermalVias
Changed lines of the file:
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@@
     (property "Reference" "R43" (id 0) (at 106.68 88.9 90))
     (property "Value" "1k" (id 1) (at 106.68 91.44 90))
-    (property "Footprint" "" (id 2) (at 106.68 95.25 0)
+    (property "Footprint" "Resistor_SMD:R_0603_1608Metric" (id 2) (at 106.68 95.25 0)
       (effects (font (size 1.27 1.27)) hide)
     )
@@
       (effects (font (size 1.27 1.27)) (justify left))
     )
-    (property "Footprint" "" (id 2) (at 111.76 111.76 0)
+    (property "Footprint" "Capacitor_SMD:C_0603_1608Metric" (id 2) (at 111.76 111.76 0)
       (effects (font (size 1.27 1.27)) hide)
     )
@@
     (property "Reference" "R44" (id 0) (at 106.68 101.6 90))
     (property "Value" "1k" (id 1) (at 106.68 104.14 90))
-    (property "Footprint" "" (id 2) (at 106.68 107.95 0)
+    (property "Footprint" "Resistor_SMD:R_0603_1608Metric" (id 2) (at 106.68 107.95 0)
       (effects (font (size 1.27 1.27)) hide)
     )
@@
     (property "Reference" "R45" (id 0) (at 106.68 120.65 90))
     (property "Value" "1k" (id 1) (at 106.68 123.19 90))
-    (property "Footprint" "" (id 2) (at 106.68 127 0)
+    (property "Footprint" "Resistor_SMD:R_0603_1608Metric" (id 2) (at 106.68 127 0)
       (effects (font (size 1.27 1.27)) hide)
     )
@@
       (effects (font (size 1.27 1.27)) (justify left))
     )
-    (property "Footprint" "" (id 2) (at 91.44 67.31 0)
+    (property "Footprint" "Resistor_SMD:R_0603_1608Metric" (id 2) (at 91.44 67.31 0)
       (effects (font (size 1.27 1.27)) hide)
     )
@@
       (effects (font (size 1.27 1.27)) (justify right))
     )
-    (property "Footprint" "" (id 2) (at 143.51 88.9 0)
+    (property "Footprint" "Capacitor_SMD:C_0603_1608Metric" (id 2) (at 143.51 88.9 0)
       (effects (font (size 1.27 1.27)) hide)
     )
@@
       (effects (font (size 1.27 1.27)) (justify right))
     )
-    (property "Footprint" "" (id 2) (at 211.328 102.87 90)
+    (property "Footprint" "Resistor_SMD:R_0603_1608Metric" (id 2) (at 211.328 102.87 90)
       (effects (font (size 1.27 1.27)) hide)
     )
@@
       (effects (font (size 1.27 1.27)) (justify left))
     )
-    (property "Footprint" "" (id 2) (at 111.76 91.44 0)
+    (property "Footprint" "Capacitor_SMD:C_0603_1608Metric" (id 2) (at 111.76 91.44 0)
       (effects (font (size 1.27 1.27)) hide)
     )
@@
     (property "Reference" "R40" (id 0) (at 106.68 57.15 90))
     (property "Value" "1k" (id 1) (at 106.68 59.69 90))
-    (property "Footprint" "" (id 2) (at 106.68 63.5 0)
+    (property "Footprint" "Resistor_SMD:R_0603_1608Metric" (id 2) (at 106.68 63.5 0)
       (effects (font (size 1.27 1.27)) hide)
     )
@@
       (effects (font (size 1.27 1.27)) (justify left))
     )
-    (property "Footprint" "" (id 2) (at 111.76 67.31 0)
+    (property "Footprint" "Capacitor_SMD:C_0603_1608Metric" (id 2) (at 111.76 67.31 0)
       (effects (font (size 1.27 1.27)) hide)
     )
@@
       (effects (font (size 1.27 1.27)) (justify left))
     )
-    (property "Footprint" "" (id 2) (at 91.44 91.44 0)
+    (property "Footprint" "Resistor_SMD:R_0603_1608Metric" (id 2) (at 91.44 91.44 0)
       (effects (font (size 1.27 1.27)) hide)
     )
@@
     (property "Reference" "Patch2" (id 0) (at 83.3628 95.885 0))
     (property "Value" "~" (id 1) (at 83.3628 93.5736 0))
-    (property "Footprint" "" (id 2) (at 81.28 90.17 0)
+    (property "Footprint" "TerminalBlock_TE-Connectivity:TerminalBlock_TE_282834-2_1x02_P2.54mm_Horizontal" (id 2) (at 81.28 90.17 0)
       (effects (font (size 1.27 1.27)) hide)
     )
@@
     (property "Reference" "R41" (id 0) (at 106.68 64.77 90))
     (property "Value" "1k" (id 1) (at 106.68 67.31 90))
-    (property "Footprint" "" (id 2) (at 106.68 71.12 0)
+    (property "Footprint" "Resistor_SMD:R_0603_1608Metric" (id 2) (at 106.68 71.12 0)
       (effects (font (size 1.27 1.27)) hide)
     )
@@
     (property "Reference" "Patch1" (id 0) (at 83.3628 71.755 0))
     (property "Value" "~" (id 1) (at 83.3628 69.4436 0))
-    (property "Footprint" "" (id 2) (at 81.28 66.04 0)
+    (property "Footprint" "TerminalBlock_TE-Connectivity:TerminalBlock_TE_282834-2_1x02_P2.54mm_Horizontal" (id 2) (at 81.28 66.04 0)
       (effects (font (size 1.27 1.27)) hide)
     )
@@
       (effects (font (size 1.27 1.27)) (justify right))
     )
-    (property "Footprint" "" (id 2) (at 201.93 83.82 0)
+    (property "Footprint" "Capacitor_SMD:C_0603_1608Metric" (id 2) (at 201.93 83.82 0)
       (effects (font (size 1.27 1.27)) hide)
     )
@@
     (property "Reference" "C36" (id 0) (at 193.0336 83.82 90))
     (property "Value" "220nF" (id 1) (at 193.0336 86.36 90))
-    (property "Footprint" "" (id 2) (at 193.04 90.17 0)
+    (property "Footprint" "Capacitor_SMD:C_0603_1608Metric" (id 2) (at 193.04 90.17 0)
       (effects (font (size 1.27 1.27)) hide)
     )
@@
     (in_bom yes) (on_board yes) (fields_autoplaced)
     (property "Reference" "U8" (id 0) (at 175.26 78.74 0))
-    (property "Value" "" (id 1) (at 175.26 81.28 0))
-    (property "Footprint" "" (id 2) (at 170.18 95.25 0)
+    (property "Value" "ADS131M04" (id 1) (at 175.26 81.28 0))
+    (property "Footprint" "Package_DFN_QFN:WQFN-20-1EP_3x3mm_P0.4mm_EP1.7x1.7mm_ThermalVias" (id 2) (at 170.18 95.25 0)
       (effects (font (size 1.27 1.27)) hide)
     )
@@
       (effects (font (size 1.27 1.27)) (justify left))
     )
-    (property "Footprint" "" (id 2) (at 111.76 130.81 0)
+    (property "Footprint" "Capacitor_SMD:C_0603_1608Metric" (id 2) (at 111.76 130.81 0)
       (effects (font (size 1.27 1.27)) hide)
     )
@@
     (property "Reference" "R42" (id 0) (at 106.68 81.28 90))
     (property "Value" "1k" (id 1) (at 106.68 83.82 90))
-    (property "Footprint" "" (id 2) (at 106.68 87.63 0)
-      (effects (font (size 1.27 1.27)) hide)
-    )
+    (property "Footprint" "Resistor_SMD:R_0603_1608Metric" (id 2) (at 106.68 87.63 0)
+      (effects (font (size 1.27 1.27)) hide)
+    )
